File: pcb/smolhhkb.kicad_pcb (KiCad board)
At the start: 4 copper layers, 228.6 x 76.2 mm, 103 parts, among them J1 USB_C, SW1 SW_Push, U1 STM32F072CBT6, U3 XC6206, U4 USBLC6-2SC6

Commit message: Fine tuning silkscreen placement
Parts:
- moved G*** 1.50 mm to (235.9, 94.4)
Routing:
- removed copper zone on B.Cu, net GND
- removed copper zone on F.Cu, net GND
- removed copper zone on F.Cu, net VBUS
